Commit message: Changed some package locations to point to jackal exploration

File: urdf/jackal.urdf.xacro (robot description, xacro)
@@ -173,5 +173,5 @@
   <xacro:include filename="$(find jackal_description)/urdf/accessories.urdf.xacro" />
   <!-- Velodyne URDF, plugin, etc -->
-  <xacro:include filename="$(find velodyne_description)/urdf/VLP-16.urdf.xacro"/>
+  <xacro:include filename="$(find jackal_exploration)/urdf/VLP-16.urdf.xacro"/>
   <VLP-16 parent="front_mount" name="velodyne" topic="/velodyne_points">
     <origin xyz="0 0 0.052" rpy="0 0 0" />
@@ -182,5 +182,5 @@
       <origin xyz="0 0 0" rpy="0.0 0.0 0.0" />
       <geometry>
-        <mesh filename="package://velodyne_description/meshes/velodyne_mount.stl"/>
+        <mesh filename="package://jackal_exploration/urdf/velodyne_mount.stl"/>
       </geometry>
       <material name="aluminum" >
